File: MagnetBoard/djshield2.brd (EAGLE design)
At the start: 5 parts

Commit message: 板子可以work, 可是 Spec 差蠻多
Parts:
- added 24V, GND, PWM, VOUT: (no value), con-molex:87758-0216
- C2: value 470u50v -> 330uF100v; device resistor:E1,8-4 -> rcl:E35-18
- moved C2 132.6 mm to (104.1, 64.8), turned to 271 degrees
- moved D1 123.9 mm to (80.0, 77.5), turned to 270 degrees
- moved C1 101.1 mm to (57.1, 81.3), turned to 359.2 degrees
- moved 30N06L 81.5 mm to (59.7, 52.1), turned to 180 degrees
- moved R1 51.7 mm to (45.7, 72.4), turned to 270 degrees
Connections:
- removed net +UB: C2.+, D1.C
- removed net -UB: 30N06L.2, C2.-, D1.A
- removed net GND: 30N06L.1, C1.-
- new net N$1: 30N06L.1, C1.-, GND.1, GND.2
- new net N$2: 30N06L.2, C2.-, D1.A, VOUT.1
- new net N$3: 24V.2, C2.+, D1.C, VOUT.2
- net N$10: now also PWM.1
Routing:
- net N$2: track 0.00 -> 126.7 mm
- net N$3: track 0.00 -> 51.6 mm
- net GND: track 41.3 -> 0.00 mm
- net N$8: track 0.00 -> 36.0 mm
- net N$10: track 0.00 -> 21.4 mm
- net N$1: track 61.9 -> 56.4 mm
- removed copper zone on layer 16, net GND
Other:
- board outline added: 160 x 100 mm
