File: MagnetBoard/djshield2.sch (EAGLE design)
At the start: 5 parts

Commit message: 板子可以work, 可是 Spec 差蠻多
Parts:
- added 24V, GND, PWM, VOUT: 87758-0216, con-molex:87758-0216
- C2: value 470u50v -> 330uF100v; device resistor:CPOL-USE1.8-4 -> rcl:CPOL-USE35-18AXIAL
Connections:
- removed net +UB: C2.+, D1.C
- removed net -UB: 30N06L.C, C2.-, D1.A
- removed net GND: 30N06L.E, C1.-
- new net N$1: 30N06L.E, C1.-, GND-1.S, GND-2.S
- new net N$2: 30N06L.C, C2.-, D1.A, VOUT-1.S
- new net N$3: 24V-2.S, C2.+, D1.C, VOUT-2.S
- net N$10: now also PWM-1.S
Changed lines of the file:
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@@
 </classes>
 <parts>
-<part name="GND7" library="SparkFun" deviceset="GND" device=""/>
 <part name="FRAME1" library="frames" deviceset="A4L-LOC" device=""/>
 <part name="R1" library="resistor-power" deviceset="R" device="RS1/4" value="500"/>
 <part name="C1" library="resistor" deviceset="CPOL-US" device="E1.8-4" value="4.7u50v"/>
 <part name="30N06L" library="transistor" deviceset="*-NPN-" device="TO126"/>
-<part name="C2" library="resistor" deviceset="CPOL-US" device="E1.8-4" value="470u50v"/>
 <part name="D1" library="diode" deviceset="1N4004" device=""/>
-<part name="SUPPLY1" library="supply2" deviceset="+24V" device=""/>
-<part name="SUPPLY2" library="supply2" deviceset="-UB" device=""/>
-<part name="SUPPLY3" library="supply2" deviceset="+UB" device=""/>
-<part name="SUPPLY4" library="supply2" deviceset="V--&gt;" device=""/>
+<part name="C2" library="rcl" deviceset="CPOL-US" device="E35-18AXIAL" value="330uF100v"/>
+<part name="24V" library="con-molex" deviceset="87758-0216" device="" value=""/>
+<part name="GND" library="con-molex" deviceset="87758-0216" device="" value=""/>
+<part name="PWM" library="con-molex" deviceset="87758-0216" device="" value=""/>
+<part name="VOUT" library="con-molex" deviceset="87758-0216" device="" value=""/>
 </parts>
 <sheets>
@@
 </plain>
 <instances>
-<instance part="GND7" gate="1" x="261.62" y="71.12"/>
 <instance part="FRAME1" gate="G$1" x="139.7" y="-7.62"/>
 <instance part="R1" gate="G$1" x="223.52" y="104.14"/>
 <instance part="C1" gate="G$1" x="238.76" y="91.44"/>
 <instance part="30N06L" gate="G$1" x="259.08" y="104.14"/>
+<instance part="D1" gate="1" x="294.64" y="96.52" rot="R270"/>
 <instance part="C2" gate="G$1" x="281.94" y="96.52" rot="R180"/>
-<instance part="D1" gate="1" x="294.64" y="96.52" rot="R270"/>
-<instance part="SUPPLY1" gate="+24V" x="281.94" y="73.66" rot="R180"/>
-<instance part="SUPPLY2" gate="G$1" x="317.5" y="109.22" rot="R90"/>
-<instance part="SUPPLY3" gate="G$1" x="317.5" y="83.82" rot="R270"/>
-<instance part="SUPPLY4" gate="G$1" x="195.58" y="104.14"/>
+<instance part="24V" gate="-2" x="281.94" y="68.58" rot="R270"/>
+<instance part="GND" gate="-1" x="261.62" y="68.58" rot="R270"/>
+<instance part="GND" gate="-2" x="271.78" y="68.58" rot="R270"/>
+<instance part="PWM" gate="-1" x="208.28" y="104.14" rot="R180"/>
+<instance part="VOUT" gate="-1" x="317.5" y="109.22"/>
+<instance part="VOUT" gate="-2" x="317.5" y="83.82"/>
 </instances>
 <busses>
 </busses>
 <nets>
-<net name="GND" class="1">
-<segment>
-<pinref part="30N06L" gate="G$1" pin="E"/>
-<pinref part="GND7" gate="1" pin="GND"/>
-<wire x1="261.62" y1="99.06" x2="261.62" y2="86.36" width="0.1524" layer="91"/>
-<pinref part="C1" gate="G$1" pin="-"/>
-<wire x1="261.62" y1="86.36" x2="261.62" y2="73.66" width="0.1524" layer="91"/>
-<wire x1="238.76" y1="86.36" x2="261.62" y2="86.36" width="0.1524" layer="91"/>
-<junction x="261.62" y="86.36"/>
-</segment>
-</net>
 <net name="N$8" class="0">
 <segment>
@@
 </segment>
 </net>
-<net name="+UB" class="0">
-<segment>
-<pinref part="C2" gate="G$1" pin="+"/>
-<wire x1="281.94" y1="93.98" x2="281.94" y2="83.82" width="0.1524" layer="91"/>
-<pinref part="SUPPLY3" gate="G$1" pin="+UB"/>
-<wire x1="281.94" y1="83.82" x2="294.64" y2="83.82" width="0.1524" layer="91"/>
-<pinref part="D1" gate="1" pin="C"/>
-<wire x1="314.96" y1="83.82" x2="294.64" y2="83.82" width="0.1524" layer="91"/>
-<wire x1="294.64" y1="83.82" x2="294.64" y2="93.98" width="0.1524" layer="91"/>
-<junction x="294.64" y="83.82"/>
-<pinref part="SUPPLY1" gate="+24V" pin="+24V"/>
-<wire x1="281.94" y1="76.2" x2="281.94" y2="83.82" width="0.1524" layer="91"/>
-<junction x="281.94" y="83.82"/>
-</segment>
-</net>
-<net name="-UB" class="0">
-<segment>
-<pinref part="D1" gate="1" pin="A"/>
-<wire x1="294.64" y1="109.22" x2="294.64" y2="99.06" width="0.1524" layer="91"/>
-<pinref part="30N06L" gate="G$1" pin="C"/>
-<wire x1="261.62" y1="109.22" x2="281.94" y2="109.22" width="0.1524" layer="91"/>
-<pinref part="C2" gate="G$1" pin="-"/>
-<wire x1="294.64" y1="109.22" x2="281.94" y2="109.22" width="0.1524" layer="91"/>
-<wire x1="281.94" y1="109.22" x2="281.94" y2="101.6" width="0.1524" layer="91"/>
-<junction x="281.94" y="109.22"/>
-<pinref part="SUPPLY2" gate="G$1" pin="-UB"/>
-<wire x1="294.64" y1="109.22" x2="314.96" y2="109.22" width="0.1524" layer="91"/>
-<junction x="294.64" y="109.22"/>
-</segment>
-</net>
 <net name="N$10" class="1">
 <segment>
 <pinref part="R1" gate="G$1" pin="1"/>
 <wire x1="210.82" y1="104.14" x2="218.44" y2="104.14" width="0.1524" layer="91"/>
+<pinref part="PWM" gate="-1" pin="S"/>
 </segment>
 </net>
+<net name="N$1" class="1">
+<segment>
+<wire x1="271.78" y1="83.82" x2="261.62" y2="83.82" width="0.1524" layer="91"/>
+<pinref part="C1" gate="G$1" pin="-"/>
+<wire x1="261.62" y1="83.82" x2="238.76" y2="83.82" width="0.1524" layer="91"/>
+<wire x1="238.76" y1="83.82" x2="238.76" y2="86.36" width="0.1524" layer="91"/>
+<pinref part="GND" gate="-2" pin="S"/>
+<wire x1="271.78" y1="83.82" x2="271.78" y2="71.12" width="0.1524" layer="91"/>
+<pinref part="30N06L" gate="G$1" pin="E"/>
+<pinref part="GND" gate="-1" pin="S"/>
+<wire x1="261.62" y1="99.06" x2="261.62" y2="83.82" width="0.1524" layer="91"/>
+<junction x="261.62" y="83.82"/>
+<wire x1="261.62" y1="83.82" x2="261.62" y2="71.12" width="0.1524" layer="91"/>
+</segment>
+</net>
+<net name="N$2" class="0">
+<segment>
+<pinref part="30N06L" gate="G$1" pin="C"/>
+<wire x1="261.62" y1="109.22" x2="281.94" y2="109.22" width="0.1524" layer="91"/>
+<pinref part="VOUT" gate="-1" pin="S"/>
+<pinref part="C2" gate="G$1" pin="-"/>
+<wire x1="281.94" y1="109.22" x2="294.64" y2="109.22" width="0.1524" layer="91"/>
+<wire x1="294.64" y1="109.22" x2="314.96" y2="109.22" width="0.1524" layer="91"/>
+<wire x1="281.94" y1="109.22" x2="281.94" y2="101.6" width="0.1524" layer="91"/>
+<pinref part="D1" gate="1" pin="A"/>
+<wire x1="294.64" y1="109.22" x2="294.64" y2="99.06" width="0.1524" layer="91"/>
+<junction x="281.94" y="109.22"/>
+<junction x="294.64" y="109.22"/>
+</segment>
+</net>
+<net name="N$3" class="0">
+<segment>
+<pinref part="D1" gate="1" pin="C"/>
+<wire x1="314.96" y1="83.82" x2="294.64" y2="83.82" width="0.1524" layer="91"/>
+<wire x1="294.64" y1="83.82" x2="294.64" y2="93.98" width="0.1524" layer="91"/>
+<pinref part="VOUT" gate="-2" pin="S"/>
+<wire x1="294.64" y1="83.82" x2="281.94" y2="83.82" width="0.1524" layer="91"/>
+<junction x="294.64" y="83.82"/>
+<pinref part="C2" gate="G$1" pin="+"/>
+<wire x1="281.94" y1="71.12" x2="281.94" y2="83.82" width="0.1524" layer="91"/>
+<pinref part="24V" gate="-2" pin="S"/>
+<junction x="281.94" y="83.82"/>
+<wire x1="281.94" y1="83.82" x2="281.94" y2="93.98" width="0.1524" layer="91"/>
+</segment>
+</net>
